Commit message: URDF simplification

File: description/omni_boat/control.xacro (robot description, xacro)
@@ -2,5 +2,5 @@
 <ros2_control name="omni_control" type="system">
   <hardware>
-    <plugin>mhseals_hardware/MavrosActuator</plugin>
+    <plugin>mhseals_control/MavrosActuator</plugin>
   </hardware>
   <joint name="front_left_thruster_joint">

File: description/omni_boat/omni_boat.xacro (robot description, xacro)
@@ -64,14 +64,5 @@
   </joint>
   <!-- ================= SENSORS ================= -->
-  <link name="gps_link">
-    <visual>
-      <origin xyz="0 0 0" rpy="0 0 0"/>
-      <material name="Material"/>
-      <geometry>
-        <mesh filename="${mesh_root}/Here3.stl"
-              scale="0.001 0.001 0.001"/>
-      </geometry>
-    </visual>
-  </link>
+  <link name="gps_link"/>
   <joint name="gps_link_joint" type="fixed">
     <parent link="base_link"/>
@@ -118,9 +109,16 @@
   <!-- ================= HULLS ================= -->
   <link name="left_hull_link">
+    <collision>
+      <origin xyz="-0.00031 0 0" rpy="0 0 0"/>
+      <geometry>
+        <mesh filename="${mesh_root}/HullCollision.stl"
+              scale="0.001 0.001 0.001"/>
+      </geometry>
+    </collision>
     <visual>
       <material name="WaterproofedHull"/>
       <origin xyz="-0.00031 0 0" rpy="0 0 0"/>
       <geometry>
-        <mesh filename="${mesh_root}/OmniHull.stl"
+        <mesh filename="${mesh_root}/HullVisual.stl"
               scale="0.001 0.001 0.001"/>
       </geometry>
@@ -133,9 +131,16 @@
   </joint>
   <link name="right_hull_link">
+    <collision>
+      <origin xyz="0.00002 0 0" rpy="0 0 0"/>
+      <geometry>
+        <mesh filename="${mesh_root}/HullCollision.stl"
+              scale="0.001 0.001 0.001"/>
+      </geometry>
+    </collision>
     <visual>
       <material name="WaterproofedHull"/>
       <origin xyz="0.00002 0 0" rpy="0 0 0"/>
       <geometry>
-        <mesh filename="${mesh_root}/OmniHull.001.stl"
+        <mesh filename="${mesh_root}/HullVisual.stl"
               scale="0.001 0.001 0.001"/>
       </geometry>
@@ -160,6 +165,6 @@
     xyz="-0.00031 -0.27970 -0.20016"
     rpy="-1.57080 0 -2.35619"
-    thruster_mesh="${mesh_root}/T200Thruster.001.stl"
-    prop_mesh="${mesh_root}/T200Propeller.001.stl"/>
+    thruster_mesh="${mesh_root}/T200Thruster.stl"
+    prop_mesh="${mesh_root}/T200Propeller.stl"/>
   <xacro:t200_thruster
     name="front_right"
@@ -167,6 +172,6 @@
     xyz="0.00002 0.27985 -0.20016"
     rpy="-1.57080 0 0.78540"
-    thruster_mesh="${mesh_root}/T200Thruster.002.stl"
-    prop_mesh="${mesh_root}/T200Propeller.002.stl"/>
+    thruster_mesh="${mesh_root}/T200Thruster.stl"
+    prop_mesh="${mesh_root}/T200Propeller.stl"/>
   <xacro:t200_thruster
     name="rear_right"
@@ -174,6 +179,6 @@
     xyz="0.00002 -0.27970 -0.20016"
     rpy="-1.57080 0 2.35619"
-    thruster_mesh="${mesh_root}/T200Thruster.003.stl"
-    prop_mesh="${mesh_root}/T200Propeller.003.stl"/>
+    thruster_mesh="${mesh_root}/T200Thruster.stl"
+    prop_mesh="${mesh_root}/T200Propeller.stl"/>
   <!-- ================= MATERIALS ================= -->
   <material name="Aluminum"><color rgba="0.64 0.64 0.64 1"/></material>

File: description/omni_boat/t200_thruster.xacro (robot description, xacro)
@@ -31,4 +31,7 @@
       <child link="${name}_thruster_link"/>
       <origin xyz="${xyz}" rpy="${rpy}"/>
+      <ros2_control>
+        <param name="thruster">true</param>
+      </ros2_control>
     </joint>
     <!-- Propeller -->
