Commit message: Fix urdf configuration

File: description/omni_boat/omni_boat.xacro (robot description, xacro)
@@ -1,11 +1,11 @@
 <?xml version="1.0"?>
 <robot name="omni_boat" xmlns:xacro="http://www.ros.org/wiki/xacro">
-  <xacro:include filename="t200_thruster.xacro"/>
-  <xacro:property name="mesh_root"
-                  value="package://mhseals_nav/description/omni_boat/meshes"/>
+  <!-- ================= INCLUDES ================= -->
+  <xacro:include filename="$(find mhseals_nav)/description/omni_boat/t200_thruster.xacro"/>
+  <xacro:property name="mesh_root" value="package://mhseals_nav/description/omni_boat/meshes"/>
   <!-- ================= BASE ================= -->
   <link name="base_link">
     <collision>
-      <origin xyz="0 0 0.02680"/>
+      <origin xyz="0 0 0.02680" rpy="0 0 -1.57080"/>
       <geometry>
         <box size="0.42126 0.36402 0.21093"/>
@@ -13,5 +13,5 @@
     </collision>
     <collision>
-      <origin xyz="0.00025 0.00008 -0.09151"/>
+      <origin xyz="0.00008 -0.00025 -0.09151" rpy="0 0 -1.57080"/>
       <geometry>
         <box size="0.43525 0.45570 0.02168"/>
@@ -20,5 +20,5 @@
     <inertial>
       <mass value="4.0"/>
-      <origin xyz="0 0 0"/>
+      <origin xyz="0 0 0" rpy="0 0 0"/>
       <inertia
         ixx="0.08480" ixy="0" ixz="0"
@@ -28,5 +28,5 @@
     <visual>
       <material name="ElectricalBox"/>
-      <origin xyz="0 0 -0.07877" rpy="1.5708 0 0"/>
+      <origin xyz="0 0 -0.07877" rpy="1.57080 0 -1.57080"/>
       <geometry>
         <mesh filename="${mesh_root}/IP65.stl"
@@ -36,5 +36,5 @@
     <visual>
       <material name="Aluminum"/>
-      <origin xyz="0 0.00008 -0.08989"/>
+      <origin xyz="0.00008 0 -0.08989" rpy="0 0 -1.57080"/>
       <geometry>
         <mesh filename="${mesh_root}/ElectricalMountFrame.stl"
@@ -46,4 +46,5 @@
   <link name="sensor_rail_link">
     <visual>
+      <origin xyz="0 0 0" rpy="0 0 0"/>
       <material name="Aluminum"/>
       <geometry>
@@ -51,13 +52,19 @@
       </geometry>
     </visual>
+    <inertial>
+      <mass value="0.8"/>
+      <origin xyz="0 0 0" rpy="0 0 0"/>
+      <inertia ixx="0.00006" ixy="0" ixz="0" iyy="0.01292" iyz="0" izz="0.01292"/>
+    </inertial>
   </link>
   <joint name="sensor_rail_link_joint" type="fixed">
     <parent link="base_link"/>
     <child link="sensor_rail_link"/>
-    <origin xyz="0 0.37825 -0.09151"/>
+    <origin xyz="0.37825 0 -0.09151" rpy="0 0 -1.57080"/>
   </joint>
   <!-- ================= SENSORS ================= -->
   <link name="gps_link">
     <visual>
+      <origin xyz="0 0 0" rpy="0 0 0"/>
       <material name="Material"/>
       <geometry>
@@ -70,5 +77,5 @@
     <parent link="base_link"/>
     <child link="gps_link"/>
-    <origin xyz="0 0.12529 0.23439"/>
+    <origin xyz="0 0 0" rpy="0 0 -1.57080"/>
   </joint>
   <link name="imu_link"/>
@@ -76,7 +83,9 @@
     <parent link="base_link"/>
     <child link="imu_link"/>
+    <origin xyz="0 0 0" rpy="0 0 -1.57080"/>
   </joint>
   <link name="camera_link">
     <visual>
+      <origin xyz="0 0 0" rpy="0 0 0"/>
       <material name="Camera"/>
       <geometry>
@@ -89,5 +98,5 @@
     <parent link="sensor_rail_link"/>
     <child link="camera_link"/>
-    <origin xyz="0 0 -0.02610"/>
+    <origin xyz="0 0 -0.02610" rpy="0 0 0"/>
   </joint>
   <link name="lidar_link">
@@ -95,5 +104,5 @@
       <material name="Lidar"/>
       <origin xyz="0.00003 -0.00061 0.03534"
-              rpy="1.5708 0 -1.5708"/>
+              rpy="1.57080 0 -1.57080"/>
       <geometry>
         <mesh filename="${mesh_root}/VelodyneVLP16.stl"
@@ -105,5 +114,5 @@
     <parent link="sensor_rail_link"/>
     <child link="lidar_link"/>
-    <origin xyz="0 0 0.01075"/>
+    <origin xyz="0 0 0.01075" rpy="0 0 0"/>
   </joint>
   <!-- ================= HULLS ================= -->
@@ -111,4 +120,5 @@
     <visual>
       <material name="WaterproofedHull"/>
+      <origin xyz="-0.00031 0 0" rpy="0 0 0"/>
       <geometry>
         <mesh filename="${mesh_root}/OmniHull.stl"
@@ -120,9 +130,10 @@
     <parent link="base_link"/>
     <child link="left_hull_link"/>
-    <origin xyz="-0.33137 -0.00008 -0.20009"/>
+    <origin xyz="-0.00008 0.33137 -0.20009" rpy="0 0 -1.57080"/>
   </joint>
   <link name="right_hull_link">
     <visual>
       <material name="WaterproofedHull"/>
+      <origin xyz="0.00002 0 0" rpy="0 0 0"/>
       <geometry>
         <mesh filename="${mesh_root}/OmniHull.001.stl"
@@ -134,5 +145,5 @@
     <parent link="base_link"/>
     <child link="right_hull_link"/>
-    <origin xyz="0.33137 -0.00008 -0.20009"/>
+    <origin xyz="-0.00008 -0.33137 -0.20009" rpy="0 0 -1.57080"/>
   </joint>
   <!-- ================= THRUSTERS ================= -->
@@ -141,26 +152,26 @@
     parent="left_hull_link"
     xyz="-0.00031 0.27985 -0.20016"
-    rpy="-1.5708 0 0.7854"
+    rpy="-1.57080 0 -0.78540"
     thruster_mesh="${mesh_root}/T200Thruster.stl"
-    prop_mesh="${mesh_root}/T200Propeller.001.stl"/>
+    prop_mesh="${mesh_root}/T200Propeller.stl"/>
   <xacro:t200_thruster
     name="rear_left"
     parent="left_hull_link"
     xyz="-0.00031 -0.27970 -0.20016"
-    rpy="-1.5708 0 2.35619"
-    thruster_mesh="${mesh_root}/T200Thruster.002.stl"
-    prop_mesh="${mesh_root}/T200Propeller.002.stl"/>
+    rpy="-1.57080 0 -2.35619"
+    thruster_mesh="${mesh_root}/T200Thruster.001.stl"
+    prop_mesh="${mesh_root}/T200Propeller.001.stl"/>
   <xacro:t200_thruster
     name="front_right"
     parent="right_hull_link"
     xyz="0.00002 0.27985 -0.20016"
-    rpy="-1.5708 0 -0.7854"
-    thruster_mesh="${mesh_root}/T200Thruster.001.stl"
-    prop_mesh="${mesh_root}/T200Propeller.stl"/>
+    rpy="-1.57080 0 0.78540"
+    thruster_mesh="${mesh_root}/T200Thruster.002.stl"
+    prop_mesh="${mesh_root}/T200Propeller.002.stl"/>
   <xacro:t200_thruster
     name="rear_right"
     parent="right_hull_link"
     xyz="0.00002 -0.27970 -0.20016"
-    rpy="-1.5708 0 -2.35619"
+    rpy="-1.57080 0 2.35619"
     thruster_mesh="${mesh_root}/T200Thruster.003.stl"
     prop_mesh="${mesh_root}/T200Propeller.003.stl"/>
@@ -168,9 +179,7 @@
   <material name="Aluminum"><color rgba="0.64 0.64 0.64 1"/></material>
   <material name="ElectricalBox"><color rgba="0.19 0.19 0.19 1"/></material>
-  <material name="Thruster"><color rgba="0.0039 0.0039 0.0039 1"/></material>
-  <material name="Propeller"><color rgba="0.0745 0.1725 0.8 1"/></material>
-  <material name="WaterproofedHull"><color rgba="0.0667 0.0667 0.0667 1"/></material>
-  <material name="Camera"><color rgba="0.15 0.15 0.15 1"/></material>
-  <material name="Lidar"><color rgba="0.01 0.22 1.0 1"/></material>
+  <material name="WaterproofedHull"><color rgba="0.06667 0.06667 0.06667 1"/></material>
+  <material name="Camera"><color rgba="0.14902 0.14902 0.14902 1"/></material>
+  <material name="Lidar"><color rgba="0.01176 0.22353 1.0 1"/></material>
   <material name="Material"><color rgba="0.02 0.02 0.02 1"/></material>
 </robot>

File: description/omni_boat/t200_thruster.xacro (robot description, xacro)
@@ -32,5 +32,5 @@
       <origin xyz="${xyz}" rpy="${rpy}"/>
     </joint>
-    <!-- Propeller (visual-only) -->
+    <!-- Propeller -->
     <link name="${name}_propeller_link">
       <visual>
@@ -42,11 +42,11 @@
       </visual>
     </link>
-    <joint name="${name}_propeller_link_joint" type="continuous">
+    <joint name="${name}_propeller_link_joint" type="fixed">
       <parent link="${name}_thruster_link"/>
       <child link="${name}_propeller_link"/>
       <origin xyz="0 0 -0.00299"/>
-      <axis xyz="0 0 1"/>
-      <limit effort="0" velocity="0"/>
     </joint>
   </xacro:macro>
+  <material name="Thruster"><color rgba="0.0039 0.0039 0.0039 1"/></material>
+  <material name="Propeller"><color rgba="0.0745 0.1725 0.8 1"/></material>
 </robot>

Commit message: Local and global odom separation

File: description/omni_boat/omni_boat.xacro (robot description, xacro)
@@ -18,12 +18,4 @@
       </geometry>
     </collision>
-    <inertial>
-      <mass value="4.0"/>
-      <origin xyz="0 0 0" rpy="0 0 0"/>
-      <inertia
-        ixx="0.08480" ixy="0" ixz="0"
-        iyy="0.09020" iyz="0"
-        izz="0.14480"/>
-    </inertial>
     <visual>
       <material name="ElectricalBox"/>

Commit message: Working local and global odometry nodes and SLAM

File: description/omni_boat/omni_boat.xacro (robot description, xacro)
@@ -35,24 +35,4 @@
     </visual>
   </link>
-  <!-- ================= SENSOR RAIL ================= -->
-  <link name="sensor_rail_link">
-    <visual>
-      <origin xyz="0 0 0" rpy="0 0 0"/>
-      <material name="Aluminum"/>
-      <geometry>
-        <box size="0.43927 0.02150 0.02150"/>
-      </geometry>
-    </visual>
-    <inertial>
-      <mass value="0.8"/>
-      <origin xyz="0 0 0" rpy="0 0 0"/>
-      <inertia ixx="0.00006" ixy="0" ixz="0" iyy="0.01292" iyz="0" izz="0.01292"/>
-    </inertial>
-  </link>
-  <joint name="sensor_rail_link_joint" type="fixed">
-    <parent link="base_link"/>
-    <child link="sensor_rail_link"/>
-    <origin xyz="0.37825 0 -0.09151" rpy="0 0 -1.57080"/>
-  </joint>
   <!-- ================= SENSORS ================= -->
   <link name="gps_link"/>
@@ -79,13 +59,12 @@
   </link>
   <joint name="camera_link_joint" type="fixed">
-    <parent link="sensor_rail_link"/>
+    <parent link="base_link"/>
     <child link="camera_link"/>
-    <origin xyz="0 0 -0.02610" rpy="0 0 0"/>
+    <origin xyz="0.287 0 -0.061" rpy="0 0 1.57080"/>
   </joint>
   <link name="lidar_link">
     <visual>
       <material name="Lidar"/>
-      <origin xyz="0.00003 -0.00061 0.03534"
-              rpy="1.57080 0 -1.57080"/>
+      <origin xyz="0 0 0" rpy="1.57080 0 1.57080"/>
       <geometry>
         <mesh filename="${mesh_root}/VelodyneVLP16.stl"
@@ -95,7 +74,7 @@
   </link>
   <joint name="lidar_link_joint" type="fixed">
-    <parent link="sensor_rail_link"/>
+    <parent link="base_link"/>
     <child link="lidar_link"/>
-    <origin xyz="0 0 0.01075" rpy="0 0 0"/>
+    <origin xyz="0 0 0.1682" rpy="0 0 -1.57080"/>
   </joint>
   <!-- ================= HULLS ================= -->
