Commit message: Blastoise urdf sensors

File: description/blastoise/blastoise.xacro (robot description, xacro)
@@ -138,4 +138,15 @@
     <child link="lidar_link"/>
     <origin xyz="0 0.01270 0.29035" rpy="0 0 0"/>
+  </joint>
+  <link name="gps_link"/>
+  <joint name="gps_link_joint" type="fixed">
+    <parent link="base_link"/>
+    <child link="gps_link"/>
+    <origin xyz="0 0.12529 0.23439"/>
+  </joint>
+  <link name="imu_link"/>
+  <joint name="imu_link_joint" type="fixed">
+    <parent link="base_link"/>
+    <child link="imu_link"/>
   </joint>
   <!-- ================= THRUSTERS ================= -->

Commit message: Put the boat description in REP-103 axes so sensors sit forward, not to port

File: description/blastoise/blastoise.xacro (robot description, xacro)
@@ -3,16 +3,19 @@
   <xacro:include filename="$(find mhseals_nav)/description/blastoise/t200_thruster.xacro"/>
   <xacro:property name="mesh_root" value="package://mhseals_nav/description/blastoise/meshes"/>
+  <!-- base_link is REP-103: x forward, y to port, z up. The meshes and the hull links are
+       in the CAD's axes (x to starboard, y forward), so they are yawed -90 degrees here;
+       sensor frames stay aligned with base_link. -->
   <!-- ================= BASE ================= -->
   <link name="base_link">
     <collision name="cross_bar_collision">
       <origin xyz="0 0 -0.01909" rpy="0 0 0"/>
-      <geometry><box size="0.43826 0.63446 0.02435"/></geometry>
+      <geometry><box size="0.63446 0.43826 0.02435"/></geometry>
     </collision>
     <collision name="ee_box_collision">
       <origin xyz="0 0 0.06988" rpy="0 0 0"/>
-      <geometry><box size="0.43980 0.50929 0.17333"/></geometry>
+      <geometry><box size="0.50929 0.43980 0.17333"/></geometry>
     </collision>
     <collision name="head_collision">
-      <origin xyz="0 -0.36901 0.00696" rpy="0 0 0"/>
+      <origin xyz="-0.36901 0 0.00696" rpy="0 0 0"/>
       <geometry><box size="0.18120 0.18120 0.18120"/></geometry>
     </collision>
@@ -25,15 +28,15 @@
     </inertial>
     <visual>
-      <origin xyz="0.24219 -0.33878 0.08816" rpy="1.57080 0 0"/>
+      <origin xyz="-0.33878 -0.24219 0.08816" rpy="1.57080 0 -1.57080"/>
       <geometry><mesh filename="${mesh_root}/bullet.stl"/></geometry>
       <material name="Material.016"/>
     </visual>
     <visual>
-      <origin xyz="0.00423 -0.13753 0.00871" rpy="1.57080 0 0"/>
+      <origin xyz="-0.13753 -0.00423 0.00871" rpy="1.57080 0 -1.57080"/>
       <geometry><mesh filename="${mesh_root}/cross_bar.stl"/></geometry>
       <material name="Material.020"/>
     </visual>
     <visual>
-      <origin xyz="-0.00358 -0.00221 0.07948" rpy="1.57080 0 0"/>
+      <origin xyz="-0.00221 0.00358 0.07948" rpy="1.57080 0 -1.57080"/>
       <geometry><mesh filename="${mesh_root}/ee_box.stl"/></geometry>
       <material name="Material.008"/>
@@ -65,5 +68,5 @@
     <parent link="base_link"/>
     <child link="left_hull_link"/>
-    <origin xyz="-0.33020 0 -0.08000" rpy="0 0 0"/>
+    <origin xyz="0 0.33020 -0.08000" rpy="0 0 -1.57080"/>
   </joint>
   <link name="right_hull_link">
@@ -91,5 +94,5 @@
     <parent link="base_link"/>
     <child link="right_hull_link"/>
-    <origin xyz="0.33020 0 -0.07800" rpy="0 0 0"/>
+    <origin xyz="0 -0.33020 -0.07800" rpy="0 0 -1.57080"/>
   </joint>
   <!-- ================= SENSOR MOUNT ================= -->
@@ -112,10 +115,10 @@
     <parent link="base_link"/>
     <child link="sensor_mount_link"/>
-    <origin xyz="0 0.27711 -0.01260" rpy="0 0 0"/>
+    <origin xyz="0.27711 0 -0.01260" rpy="0 0 0"/>
   </joint>
   <!-- ================= SENSORS ================= -->
   <link name="front_camera_link">
     <visual>
-      <origin xyz="0.00056 0 0" rpy="1.57080 0 0"/>
+      <origin xyz="0 -0.00056 0" rpy="1.57080 0 -1.57080"/>
       <geometry><mesh filename="${mesh_root}/front_camera.stl"/></geometry>
       <material name="Material.005"/>
@@ -125,9 +128,9 @@
     <parent link="sensor_mount_link"/>
     <child link="front_camera_link"/>
-    <origin xyz="0 0.04990 0.13779" rpy="0 0 0"/>
+    <origin xyz="0.04990 0 0.13779" rpy="0 0 0"/>
   </joint>
   <link name="lidar_link">
     <visual>
-      <origin xyz="0.00019 -0.01946 -0.01764" rpy="1.57080 0 0"/>
+      <origin xyz="-0.01946 -0.00019 -0.01764" rpy="1.57080 0 -1.57080"/>
       <geometry><mesh filename="${mesh_root}/lidar.stl"/></geometry>
       <material name="Material.003"/>
@@ -137,5 +140,5 @@
     <parent link="sensor_mount_link"/>
     <child link="lidar_link"/>
-    <origin xyz="0 0.01270 0.29035" rpy="0 0 0"/>
+    <origin xyz="0.01270 0 0.29035" rpy="0 0 0"/>
   </joint>
   <link name="gps_link"/>
@@ -143,5 +146,5 @@
     <parent link="base_link"/>
     <child link="gps_link"/>
-    <origin xyz="0 0.12529 0.23439"/>
+    <origin xyz="0.12529 0 0.23439"/>
   </joint>
   <link name="imu_link"/>

Commit message: Give the blastoise links physical inertias at crane_ml's 30 kg and mark mass and CoM as unmeasured
Every link carried a 1e-3 placeholder tensor (composite Iyy 0.31 kg m^2, impossible for two
1.06 m hulls). Each tensor is now its link's solid box or cylinder; the composite yaw inertia
is about 4.5 kg m^2 against crane_ml's 4.1. Frames are unchanged; only TF reads this file.

File: description/blastoise/blastoise.xacro (robot description, xacro)
@@ -20,10 +20,15 @@
       <geometry><box size="0.18120 0.18120 0.18120"/></geometry>
     </collision>
+    <!-- Mass and CoM are NOT measured: the boat has not been weighed. The links add up to
+         crane_ml's 30 kg "loaded" (deck, electronics and batteries 10 kg here, hulls 9 kg each,
+         mount 0.3, thrusters 4 x 0.427) with the CoM at base_link; each tensor is the solid box
+         (or cylinder) of its link, so the composite yaw inertia is about 4.5 kg m^2. Only TF reads
+         this file at runtime; replace the numbers once the boat is weighed and balanced. -->
     <inertial>
-      <mass value="3.0"/>
+      <mass value="10.0"/>
       <origin xyz="0 0 0" rpy="0 0 0"/>
-      <inertia ixx="0.001" ixy="0" ixz="0"
-               iyy="0.001" iyz="0"
-               izz="0.001"/>
+      <inertia ixx="0.195" ixy="0" ixz="0"
+               iyy="0.364" iyz="0"
+               izz="0.492"/>
     </inertial>
     <visual>
@@ -52,10 +57,10 @@
       </geometry>
     </collision>
-    <inertial>
-      <mass value="7.0"/>
+    <inertial>  <!-- 1.06 m long (link y), 0.16 m wide, 0.2 m deep slender box -->
+      <mass value="9.0"/>
       <origin xyz="0 0 0" rpy="0 0 0"/>
-      <inertia ixx="0.001" ixy="0" ixz="0"
-               iyy="0.001" iyz="0"
-               izz="0.001"/>
+      <inertia ixx="0.873" ixy="0" ixz="0"
+               iyy="0.049" iyz="0"
+               izz="0.862"/>
     </inertial>
     <visual>
@@ -78,10 +83,10 @@
       </geometry>
     </collision>
-    <inertial>
-      <mass value="7.0"/>
+    <inertial>  <!-- 1.06 m long (link y), 0.16 m wide, 0.2 m deep slender box -->
+      <mass value="9.0"/>
       <origin xyz="0 0 0" rpy="0 0 0"/>
-      <inertia ixx="0.001" ixy="0" ixz="0"
-               iyy="0.001" iyz="0"
-               izz="0.001"/>
+      <inertia ixx="0.873" ixy="0" ixz="0"
+               iyy="0.049" iyz="0"
+               izz="0.862"/>
     </inertial>
     <visual>
@@ -104,10 +109,10 @@
       </geometry>
     </collision>
-    <inertial>
+    <inertial>  <!-- the collision cylinder's centre and tensor -->
       <mass value="0.3"/>
-      <origin xyz="0 0 0" rpy="0 0 0"/>
-      <inertia ixx="0.001" ixy="0" ixz="0"
-               iyy="0.001" iyz="0"
-               izz="0.001"/>
+      <origin xyz="0 0 0.15839" rpy="0 0 0"/>
+      <inertia ixx="0.0033" ixy="0" ixz="0"
+               iyy="0.0033" iyz="0"
+               izz="0.0008"/>
     </inertial>
   </link>

Commit message: Set gps_link and imu_link to the 2026-10-25 taped offsets from the CoM: antenna (0.051, -0.127), Cube (-0.051, -0.127); the URDF is the source for GPS1_POS and INS_POS, pinned by test_sensor_offsets

File: description/blastoise/blastoise.xacro (robot description, xacro)
@@ -147,9 +147,11 @@
     <origin xyz="0.01270 0 0.29035" rpy="0 0 0"/>
   </joint>
+  <!-- Here4 antenna and CubeOrange+, taped from the CoM on 2026-10-25 (heights not measured).
+       The FCU's GPS1_POS_* and INS_POS1..3_* are these in FRD: x as is, y negated. -->
   <link name="gps_link"/>
   <joint name="gps_link_joint" type="fixed">
     <parent link="base_link"/>
     <child link="gps_link"/>
-    <origin xyz="0.12529 0 0.23439"/>
+    <origin xyz="0.051 -0.127 0.23439"/>
   </joint>
   <link name="imu_link"/>
@@ -157,4 +159,5 @@
     <parent link="base_link"/>
     <child link="imu_link"/>
+    <origin xyz="-0.051 -0.127 0"/>
   </joint>
   <!-- ================= THRUSTERS ================= -->

Commit message: ekf_local at 100 Hz on a 100 Hz ATTITUDE_QUATERNION, the ZED 2i gyro and magnetometer heading as a second yaw reference (front_imu_link in the URDF), and /gps/fix in gps_link so navsat removes the antenna lever arm (15 cm circle in a spin before, 1 cm after)

File: description/blastoise/blastoise.xacro (robot description, xacro)
@@ -134,4 +134,17 @@
     <child link="front_camera_link"/>
     <origin xyz="0.04990 0 0.13779" rpy="0 0 0"/>
+  </joint>
+  <!-- ZED 2i IMU (frame_id of /front/zed_node/imu/data and /imu/zed). front_camera_link is the
+       camera's bottom mounting screw; the ZED wrapper's own description (publish_urdf, on the
+       Orin) hangs front_camera_center 0.015 above it, unrotated for the zed2i (bottom_slope 0),
+       but it has no IMU link: the wrapper's IMU TF is off (camera.launch.py publish_imu_tf
+       false), so this is its only publisher and the ODROID's EKF needs no Orin TF for it.
+       Placed at the camera centre with the camera's axes: the SDK's factory camera-IMU
+       transform is a few mm and under a degree, which a gyro or heading does not feel. -->
+  <link name="front_imu_link"/>
+  <joint name="front_imu_joint" type="fixed">
+    <parent link="front_camera_link"/>
+    <child link="front_imu_link"/>
+    <origin xyz="0 0 0.015" rpy="0 0 0"/>
   </joint>
   <link name="lidar_link">

Commit message: Drop the ZED gyro from ekf_local (no process noise for its bias, so it led the fused yaw rate) and the magnetometer heading that shipped off; zed_imu_reference, its config, launch entry and front_imu_link go with them

File: description/blastoise/blastoise.xacro (robot description, xacro)
@@ -134,17 +134,4 @@
     <child link="front_camera_link"/>
     <origin xyz="0.04990 0 0.13779" rpy="0 0 0"/>
-  </joint>
-  <!-- ZED 2i IMU (frame_id of /front/zed_node/imu/data and /imu/zed). front_camera_link is the
-       camera's bottom mounting screw; the ZED wrapper's own description (publish_urdf, on the
-       Orin) hangs front_camera_center 0.015 above it, unrotated for the zed2i (bottom_slope 0),
-       but it has no IMU link: the wrapper's IMU TF is off (camera.launch.py publish_imu_tf
-       false), so this is its only publisher and the ODROID's EKF needs no Orin TF for it.
-       Placed at the camera centre with the camera's axes: the SDK's factory camera-IMU
-       transform is a few mm and under a degree, which a gyro or heading does not feel. -->
-  <link name="front_imu_link"/>
-  <joint name="front_imu_joint" type="fixed">
-    <parent link="front_camera_link"/>
-    <child link="front_imu_link"/>
-    <origin xyz="0 0 0.015" rpy="0 0 0"/>
   </joint>
   <link name="lidar_link">
